File: STM32F446RC/STM32F446RC2.sch (EAGLE design)
At the start: 75 parts, among them IC1 STM32F446RCT6

Commit message: version2
Parts:
- C1, C3, C4, C5, C6: value 100n+1u -> 100n
- C11, C2, C9: value 20p -> 22p
- JP4: SPICEPREFIX X -> (none)
- R3: value (none) -> 47
- renumbered C0 to JP29, C13 to JP26
Connections:
- net N$53: no longer C9.2
Other:
- moved on the sheet: C9
Changed lines of the file:
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@@
 <part name="IC1" library="STM32F446RCT6" deviceset="STM32F446RCT6" device=""/>
 <part name="R1" library="rcl" library_urn="urn:adsk.eagle:library:334" deviceset="R-US_" device="0204/2V" package3d_urn="urn:adsk.eagle:package:23495/1" value="10k"/>
-<part name="C1" library="capacitor-wima" library_urn="urn:adsk.eagle:library:116" deviceset="C" device="2,5-3" package3d_urn="urn:adsk.eagle:package:5436/1" value="100n+1u"/>
-<part name="C3" library="capacitor-wima" library_urn="urn:adsk.eagle:library:116" deviceset="C" device="2,5-3" package3d_urn="urn:adsk.eagle:package:5436/1" value="100n+1u"/>
-<part name="C4" library="capacitor-wima" library_urn="urn:adsk.eagle:library:116" deviceset="C" device="2,5-3" package3d_urn="urn:adsk.eagle:package:5436/1" value="100n+1u"/>
-<part name="C5" library="capacitor-wima" library_urn="urn:adsk.eagle:library:116" deviceset="C" device="2,5-3" package3d_urn="urn:adsk.eagle:package:5436/1" value="100n+1u"/>
-<part name="R3" library="rcl" library_urn="urn:adsk.eagle:library:334" deviceset="R-US_" device="0204/2V" package3d_urn="urn:adsk.eagle:package:23495/1"/>
-<part name="C6" library="capacitor-wima" library_urn="urn:adsk.eagle:library:116" deviceset="C" device="2,5-3" package3d_urn="urn:adsk.eagle:package:5436/1" value="100n+1u"/>
+<part name="C1" library="capacitor-wima" library_urn="urn:adsk.eagle:library:116" deviceset="C" device="2,5-3" package3d_urn="urn:adsk.eagle:package:5436/1" value="100n"/>
+<part name="C3" library="capacitor-wima" library_urn="urn:adsk.eagle:library:116" deviceset="C" device="2,5-3" package3d_urn="urn:adsk.eagle:package:5436/1" value="100n"/>
+<part name="C4" library="capacitor-wima" library_urn="urn:adsk.eagle:library:116" deviceset="C" device="2,5-3" package3d_urn="urn:adsk.eagle:package:5436/1" value="100n"/>
+<part name="C5" library="capacitor-wima" library_urn="urn:adsk.eagle:library:116" deviceset="C" device="2,5-3" package3d_urn="urn:adsk.eagle:package:5436/1" value="100n"/>
+<part name="R3" library="rcl" library_urn="urn:adsk.eagle:library:334" deviceset="R-US_" device="0204/2V" package3d_urn="urn:adsk.eagle:package:23495/1" value="47"/>
+<part name="C6" library="capacitor-wima" library_urn="urn:adsk.eagle:library:116" deviceset="C" device="2,5-3" package3d_urn="urn:adsk.eagle:package:5436/1" value="100n"/>
 <part name="C7" library="capacitor-wima" library_urn="urn:adsk.eagle:library:116" deviceset="C" device="2,5-3" package3d_urn="urn:adsk.eagle:package:5436/1" value="2.2U"/>
 <part name="C8" library="capacitor-wima" library_urn="urn:adsk.eagle:library:116" deviceset="C" device="2,5-3" package3d_urn="urn:adsk.eagle:package:5436/1" value="100n+1u"/>
-<part name="C9" library="capacitor-wima" library_urn="urn:adsk.eagle:library:116" deviceset="C" device="2,5-3" package3d_urn="urn:adsk.eagle:package:5436/1" value="20p"/>
-<part name="C11" library="capacitor-wima" library_urn="urn:adsk.eagle:library:116" deviceset="C" device="2,5-3" package3d_urn="urn:adsk.eagle:package:5436/1" value="20p"/>
+<part name="C9" library="capacitor-wima" library_urn="urn:adsk.eagle:library:116" deviceset="C" device="2,5-3" package3d_urn="urn:adsk.eagle:package:5436/1" value="22p"/>
+<part name="C11" library="capacitor-wima" library_urn="urn:adsk.eagle:library:116" deviceset="C" device="2,5-3" package3d_urn="urn:adsk.eagle:package:5436/1" value="22p"/>
 <part name="JP3" library="F405Pill" deviceset="HEADERHOLE" device="-HEADERHOLE"/>
-<part name="JP4" library="F405Pill" deviceset="HEADERHOLE" device="-HEADERHOLE">
-<attribute name="SPICEPREFIX" value="X"/>
-</part>
+<part name="JP4" library="F405Pill" deviceset="HEADERHOLE" device="-HEADERHOLE"/>
 <part name="JP5" library="F405Pill" deviceset="HEADERHOLE" device="-HEADERHOLE"/>
 <part name="JP6" library="F405Pill" deviceset="HEADERHOLE" device="-HEADERHOLE"/>
@@
 <part name="JP24" library="F405Pill" deviceset="HEADERHOLE" device="-HEADERHOLE"/>
 <part name="JP25" library="F405Pill" deviceset="HEADERHOLE" device="-HEADERHOLE"/>
-<part name="C13" library="F405Pill" deviceset="HEADERHOLE" device="-HEADERHOLE"/>
+<part name="JP26" library="F405Pill" deviceset="HEADERHOLE" device="-HEADERHOLE"/>
 <part name="JP27" library="F405Pill" deviceset="HEADERHOLE" device="-HEADERHOLE"/>
 <part name="JP28" library="F405Pill" deviceset="HEADERHOLE" device="-HEADERHOLE"/>
-<part name="C0" library="F405Pill" deviceset="HEADERHOLE" device="-HEADERHOLE"/>
+<part name="JP29" library="F405Pill" deviceset="HEADERHOLE" device="-HEADERHOLE"/>
 <part name="JP30" library="F405Pill" deviceset="HEADERHOLE" device="-HEADERHOLE"/>
 <part name="JP31" library="F405Pill" deviceset="HEADERHOLE" device="-HEADERHOLE"/>
@@
 <part name="JP65" library="F405Pill" deviceset="HEADERHOLE" device="-HEADERHOLE"/>
 <part name="JP7" library="F405Pill" deviceset="HEADERHOLE" device="-HEADERHOLE"/>
-<part name="C2" library="capacitor-wima" library_urn="urn:adsk.eagle:library:116" deviceset="C" device="2,5-3" package3d_urn="urn:adsk.eagle:package:5436/1" value="20p"/>
+<part name="C2" library="capacitor-wima" library_urn="urn:adsk.eagle:library:116" deviceset="C" device="2,5-3" package3d_urn="urn:adsk.eagle:package:5436/1" value="22p"/>
 </parts>
 <sheets>
@@
 <attribute name="VALUE" x="25.019" y="34.544" size="1.778" layer="96" rot="R90"/>
 </instance>
-<instance part="C9" gate="G$1" x="-27.94" y="66.04" rot="R90">
-<attribute name="NAME" x="-28.321" y="67.564" size="1.778" layer="95" rot="R90"/>
-<attribute name="VALUE" x="-23.241" y="67.564" size="1.778" layer="96" rot="R90"/>
+<instance part="C9" gate="G$1" x="-27.94" y="63.5" rot="R90">
+<attribute name="NAME" x="-28.321" y="65.024" size="1.778" layer="95" rot="R90"/>
+<attribute name="VALUE" x="-23.241" y="65.024" size="1.778" layer="96" rot="R90"/>
 </instance>
 <instance part="C11" gate="G$1" x="-27.94" y="55.88" rot="R90">
@@
 <attribute name="VALUE" x="83.82" y="56.388" size="0.4064" layer="96" ratio="10"/>
 </instance>
-<instance part="C13" gate="G$1" x="30.48" y="60.96">
+<instance part="JP26" gate="G$1" x="30.48" y="60.96">
 <attribute name="VALUE" x="30.48" y="60.452" size="0.4064" layer="96" ratio="10" rot="R180"/>
 </instance>
@@
 <attribute name="VALUE" x="83.82" y="46.228" size="0.4064" layer="96" ratio="10"/>
 </instance>
-<instance part="C0" gate="G$1" x="30.48" y="45.72">
+<instance part="JP29" gate="G$1" x="30.48" y="45.72">
 <attribute name="VALUE" x="30.48" y="45.212" size="0.4064" layer="96" ratio="10" rot="R180"/>
 </instance>
@@
 <segment>
 <pinref part="IC1" gate="G$1" pin="PC0"/>
-<pinref part="C0" gate="G$1" pin="P$1"/>
+<pinref part="JP29" gate="G$1" pin="P$1"/>
 </segment>
 </net>
@@
 <segment>
 <pinref part="IC1" gate="G$1" pin="PC13"/>
-<pinref part="C13" gate="G$1" pin="P$1"/>
+<pinref part="JP26" gate="G$1" pin="P$1"/>
 </segment>
 </net>
@@
 <net name="N$53" class="0">
 <segment>
-<pinref part="C9" gate="G$1" pin="2"/>
-<wire x1="-17.78" y1="66.04" x2="-22.86" y2="66.04" width="0.1524" layer="91"/>
 <pinref part="IC1" gate="G$1" pin="PH0-OSC_IN"/>
 <wire x1="30.48" y1="53.34" x2="20.32" y2="53.34" width="0.1524" layer="91"/>
@@
 <wire x1="12.7" y1="63.5" x2="-5.08" y2="63.5" width="0.1524" layer="91"/>
 <wire x1="-5.08" y1="63.5" x2="-25.4" y2="63.5" width="0.1524" layer="91"/>
-<wire x1="-17.78" y1="66.04" x2="-25.4" y2="63.5" width="0.1524" layer="91"/>
 <pinref part="C2" gate="G$1" pin="2"/>
 <junction x="-5.08" y="63.5"/>
@@
 <pinref part="C9" gate="G$1" pin="1"/>
 <wire x1="-30.48" y1="55.88" x2="-30.48" y2="60.96" width="0.1524" layer="91"/>
-<wire x1="-30.48" y1="60.96" x2="-30.48" y2="66.04" width="0.1524" layer="91"/>
+<wire x1="-30.48" y1="60.96" x2="-30.48" y2="63.5" width="0.1524" layer="91"/>
 <wire x1="-30.48" y1="60.96" x2="-33.02" y2="60.96" width="0.1524" layer="91"/>
 <junction x="-30.48" y="60.96"/>
