File: STM32F413CG/STM32F413CG.brd (EAGLE design)
At the start: 73.4 x 33 mm, 58 parts, among them IC1 STM32F413CGU6, IC2 CS43L22-CNZ, IC3 LP3985IM5-2.5, J2 1503_02, X1 USB-MICROB-SMD

Commit message: final stage
Parts:
- added C33: 100nf, capacitor-wima:C2.5-2
- added C34: 1UF, capacitor-wima:C2.5-2
- added JP10, JP5, JP6, JP7, JP8, JP9: (no value), F405Pill:1X1-HEADER-HOLE
- added MK2: MP34DT05TR-A, MP34DT05TR-A:MP34DT05TRA
- added SW1: (no value), special:EDG-01
- moved C32 5.80 mm to (15.8, 29.8)
- moved C31 5.80 mm to (13.2, 29.8)
- moved MK1 5.53 mm to (8.89, 29.0)
- moved C10 1.47 mm to (3.58, 28.9)
- moved C9 1.39 mm to (3.72, 25.8)
- moved R6 1.35 mm to (9.35, 8.25)
- moved C11 1.35 mm to (3.75, 23.1)
- moved C12 1.15 mm to (9.27, 17.7)
- moved R5 0.90 mm to (10.7, 9.83)
- moved R4 0.69 mm to (8.35, 23.1), turned to 110 degrees
- moved R2 0.45 mm to (31.8, 11.7)
- moved Q1 0.20 mm to (31.9, 16.3)
- moved JP2 0.10 mm to (6.90, 2.53)
- moved JP3 0.10 mm to (4.34, 2.53)
- moved JP4 0.07 mm to (12.0, 2.53)
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Connections:
- new net A1: IC1.11, JP8.1
- new net A2: IC1.12, JP9.1
- new net A3: IC1.13, JP10.1
- new net B12: IC1.25, JP7.1
- new net B13: IC1.26, JP6.1
- new net C14: IC1.3, IC2.32, R13.1
- new net N$2: C33.1, C34.1, MK2.3, MK2.4, SW1.1
- net A4: now also MK2.2
- net A8: now also MK2.1
- net B8: now also JP5.1; no longer IC2.32, R13.1
- net GND: now also C33.2, C34.2, MK2.5, MK2.6, MK2.7, MK2.8
- net VDD: now also SW1.2
Routing:
- net VDD: track 179.5 -> 246.2 mm, vias 2 -> 5
- net GND: track 287.2 -> 343.1 mm
- net C14: track 0.00 -> 54.9 mm, vias 0 -> 2
- net A8: track 24.9 -> 65.5 mm, vias 2 -> 4
- net A4: track 12.9 -> 41.0 mm, vias 2 -> 3
- net B13: track 0.00 -> 25.7 mm
- net B12: track 0.00 -> 21.7 mm, vias 0 -> 2
- net A1: track 0.00 -> 20.1 mm
- net B8: track 28.3 -> 8.38 mm, vias 2 -> 1
- net A2: track 0.00 -> 18.0 mm
- net A3: track 0.00 -> 16.8 mm
- net N$2: track 0.00 -> 11.2 mm, vias 0 -> 1
- net 5V: track 42.6 -> 39.2 mm
- net N$13: track 55.3 -> 57.1 mm, vias 0 -> 1
- net N$31: track 4.91 -> 6.24 mm
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