File: STM32F413CG/STM32F413CG.sch (EAGLE design)
At the start: 58 parts, among them IC1 STM32F413CGU6, IC2 CS43L22-CNZ, IC3 LP3985IM5-2.5, J2 1503_02, X1 USB-MICROB-SMD

Commit message: final stage
Parts:
- added C33: 100nf, capacitor-wima:C2.5/2
- added C34: 1UF, capacitor-wima:C2.5/2
- added JP10, JP5, JP6, JP7, JP8, JP9: (no value), F405Pill:HEADERHOLE-HEADERHOLE
- added MK2: MP34DT05TR-A, MP34DT05TR-A:MP34DT05TR-A
- added SW1: (no value), special:SW_DIP-1
Connections:
- new net A1: IC1.PA1, JP8.P$1
- new net A2: IC1.PA2, JP9.P$1
- new net A3: IC1.PA3, JP10.P$1
- new net B12: IC1.PB12, JP7.P$1
- new net B13: IC1.PB13, JP6.P$1
- new net C14: IC1.PC14-OSC32_IN, IC2.!RESET, R13.1
- new net N$2: C33.1, C34.1, MK2.LR, MK2.VDD, SW1.1
- net A4: now also MK2.DOUT
- net A8: now also MK2.CLK
- net B8: now also JP5.P$1; no longer IC2.!RESET, R13.1
- net GND: now also C33.2, C34.2, MK2.GND_1, MK2.GND_2, MK2.GND_3, MK2.GND_4
- net VDD: now also SW1.2
Other:
- moved on the sheet: R2
