File: STM32F413CG/STM32F413CG_CS43L22.brd (EAGLE design)
At the start: 73.4 x 33 mm, 69 parts, among them IC1 STM32F413CGU6, IC2 CS43L22-CNZ, IC3 LP3985IM5-2.5, J2 1503_02, X1 USB-MICROB-SMD

Commit message: added
Changed lines of the file:
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@@
 <layer number="23" name="tOrigins" color="15" fill="1" visible="yes" active="yes"/>
 <layer number="24" name="bOrigins" color="15" fill="1" visible="yes" active="yes"/>
-<layer number="25" name="tNames" color="7" fill="1" visible="yes" active="yes"/>
+<layer number="25" name="tNames" color="7" fill="1" visible="no" active="yes"/>
 <layer number="26" name="bNames" color="7" fill="1" visible="no" active="yes"/>
 <layer number="27" name="tValues" color="7" fill="1" visible="no" active="yes"/>
@@
 <layer number="37" name="tTest" color="7" fill="1" visible="no" active="yes"/>
 <layer number="38" name="bTest" color="7" fill="1" visible="no" active="yes"/>
-<layer number="39" name="tKeepout" color="4" fill="11" visible="yes" active="yes"/>
-<layer number="40" name="bKeepout" color="1" fill="11" visible="yes" active="yes"/>
-<layer number="41" name="tRestrict" color="4" fill="10" visible="yes" active="yes"/>
-<layer number="42" name="bRestrict" color="1" fill="10" visible="yes" active="yes"/>
-<layer number="43" name="vRestrict" color="2" fill="10" visible="yes" active="yes"/>
+<layer number="39" name="tKeepout" color="4" fill="11" visible="no" active="yes"/>
+<layer number="40" name="bKeepout" color="1" fill="11" visible="no" active="yes"/>
+<layer number="41" name="tRestrict" color="4" fill="10" visible="no" active="yes"/>
+<layer number="42" name="bRestrict" color="1" fill="10" visible="no" active="yes"/>
+<layer number="43" name="vRestrict" color="2" fill="10" visible="no" active="yes"/>
 <layer number="44" name="Drills" color="7" fill="1" visible="no" active="yes"/>
 <layer number="45" name="Holes" color="7" fill="1" visible="no" active="yes"/>
@@
 <layer number="47" name="Measures" color="7" fill="1" visible="no" active="yes"/>
 <layer number="48" name="Document" color="7" fill="1" visible="yes" active="yes"/>
-<layer number="49" name="Reference" color="7" fill="1" visible="yes" active="yes"/>
-<layer number="50" name="dxf" color="7" fill="1" visible="yes" active="yes"/>
+<layer number="49" name="Reference" color="7" fill="1" visible="no" active="yes"/>
+<layer number="50" name="dxf" color="7" fill="1" visible="no" active="yes"/>
 <layer number="51" name="tDocu" color="7" fill="1" visible="yes" active="yes"/>
-<layer number="52" name="bDocu" color="7" fill="1" visible="yes" active="yes"/>
-<layer number="53" name="tGND_GNDA" color="7" fill="1" visible="yes" active="yes"/>
-<layer number="54" name="bGND_GNDA" color="7" fill="1" visible="yes" active="yes"/>
-<layer number="56" name="wert" color="7" fill="1" visible="yes" active="yes"/>
+<layer number="52" name="bDocu" color="7" fill="1" visible="no" active="yes"/>
+<layer number="53" name="tGND_GNDA" color="7" fill="1" visible="no" active="yes"/>
+<layer number="54" name="bGND_GNDA" color="7" fill="1" visible="no" active="yes"/>
+<layer number="56" name="wert" color="7" fill="1" visible="no" active="yes"/>
 <layer number="88" name="SimResults" color="9" fill="1" visible="no" active="no"/>
 <layer number="89" name="SimProbes" color="9" fill="1" visible="no" active="no"/>
@@
 <layer number="98" name="Guide" color="6" fill="1" visible="no" active="no"/>
 <layer number="99" name="SpiceOrder" color="5" fill="1" visible="no" active="no"/>
-<layer number="100" name="Muster" color="7" fill="1" visible="yes" active="yes"/>
-<layer number="101" name="Patch_Top" color="7" fill="1" visible="yes" active="yes"/>
-<layer number="102" name="Vscore" color="7" fill="1" visible="yes" active="yes"/>
-<layer number="103" name="tMap" color="7" fill="1" visible="yes" active="yes"/>
+<layer number="100" name="Muster" color="7" fill="1" visible="no" active="yes"/>
+<layer number="101" name="Patch_Top" color="7" fill="1" visible="no" active="yes"/>
+<layer number="102" name="Vscore" color="7" fill="1" visible="no" active="yes"/>
+<layer number="103" name="tMap" color="7" fill="1" visible="no" active="yes"/>
 <layer number="104" name="Name" color="7" fill="1" visible="no" active="yes"/>
-<layer number="105" name="tPlate" color="7" fill="1" visible="yes" active="yes"/>
-<layer number="106" name="bPlate" color="7" fill="1" visible="yes" active="yes"/>
-<layer number="107" name="Crop" color="7" fill="1" visible="yes" active="yes"/>
-<layer number="116" name="Patch_BOT" color="7" fill="1" visible="yes" active="yes"/>
-<layer number="121" name="_tsilk" color="7" fill="1" visible="yes" active="yes"/>
-<layer number="122" name="_bsilk" color="7" fill="1" visible="yes" active="yes"/>
+<layer number="105" name="tPlate" color="7" fill="1" visible="no" active="yes"/>
+<layer number="106" name="bPlate" color="7" fill="1" visible="no" active="yes"/>
+<layer number="107" name="Crop" color="7" fill="1" visible="no" active="yes"/>
+<layer number="116" name="Patch_BOT" color="7" fill="1" visible="no" active="yes"/>
+<layer number="121" name="_tsilk" color="7" fill="1" visible="no" active="yes"/>
+<layer number="122" name="_bsilk" color="7" fill="1" visible="no" active="yes"/>
 <layer number="125" name="_tNames" color="7" fill="1" visible="no" active="yes"/>
 <layer number="126" name="_bNames" color="7" fill="1" visible="no" active="yes"/>
 <layer number="127" name="_tValues" color="7" fill="1" visible="no" active="yes"/>
-<layer number="128" name="_bValues" color="7" fill="1" visible="yes" active="yes"/>
+<layer number="128" name="_bValues" color="7" fill="1" visible="no" active="yes"/>
 <layer number="144" name="Drill_legend" color="7" fill="1" visible="yes" active="yes"/>
 <layer number="151" name="HeatSink" color="7" fill="1" visible="yes" active="yes"/>
@@
 </polygon>
 </signal>
-<signal name="N$12">
-<via x="40.4" y="13.35" extent="1-16" drill="0.35"/>
-</signal>
-<signal name="N$14">
-<via x="41.1" y="14.15" extent="1-16" drill="0.35"/>
-</signal>
-<signal name="N$15">
-<via x="42.35" y="14.1" extent="1-16" drill="0.35"/>
-</signal>
-<signal name="N$16">
-<via x="41.8" y="13.25" extent="1-16" drill="0.35"/>
-</signal>
-<signal name="N$17">
-<via x="40.95" y="12.45" extent="1-16" drill="0.35"/>
-</signal>
-<signal name="N$18">
-<via x="41.6" y="11.7" extent="1-16" drill="0.35"/>
-</signal>
-<signal name="N$20">
-<via x="42.3" y="12.4" extent="1-16" drill="0.35"/>
-</signal>
-<signal name="N$21">
-<via x="43" y="13.15" extent="1-16" drill="0.35"/>
-</signal>
 <signal name="HEAT2">
 <polygon width="0.254" layer="16">
@@
 </polygon>
 </signal>
+<signal name="N$12">
+<via x="17.15" y="13" extent="1-16" drill="0.35"/>
+</signal>
+<signal name="N$14">
+<via x="18.05" y="13.85" extent="1-16" drill="0.35"/>
+</signal>
+<signal name="N$15">
+<via x="19" y="14.6" extent="1-16" drill="0.35"/>
+</signal>
+<signal name="N$16">
+<via x="18.05" y="11.95" extent="1-16" drill="0.35"/>
+</signal>
+<signal name="N$17">
+<via x="19" y="12.75" extent="1-16" drill="0.35"/>
+</signal>
+<signal name="N$18">
+<via x="20.05" y="13.65" extent="1-16" drill="0.35"/>
+</signal>
+<signal name="N$20">
+<via x="21.2" y="13.05" extent="1-16" drill="0.35"/>
+</signal>
+<signal name="N$21">
+<via x="20.35" y="11.9" extent="1-16" drill="0.35"/>
+</signal>
 <signal name="N$22">
-<via x="16.75" y="12.85" extent="1-16" drill="0.35"/>
+<via x="19.3" y="11.05" extent="1-16" drill="0.35"/>
 </signal>
 <signal name="N$23">
-<via x="17.6" y="13.65" extent="1-16" drill="0.35"/>
+<via x="40.25" y="13.2" extent="1-16" drill="0.35"/>
 </signal>
 <signal name="N$24">
-<via x="18.35" y="14.5" extent="1-16" drill="0.35"/>
+<via x="40.95" y="13.95" extent="1-16" drill="0.35"/>
 </signal>
 <signal name="N$36">
-<via x="19.5" y="14.95" extent="1-16" drill="0.35"/>
+<via x="41.75" y="14.6" extent="1-16" drill="0.35"/>
 </signal>
 <signal name="N$37">
-<via x="19.1" y="13.65" extent="1-16" drill="0.35"/>
+<via x="42.55" y="13.65" extent="1-16" drill="0.35"/>
 </signal>
 <signal name="N$39">
-<via x="18.35" y="12.75" extent="1-16" drill="0.35"/>
+<via x="41.6" y="13.2" extent="1-16" drill="0.35"/>
 </signal>
 <signal name="N$40">
-<via x="17.95" y="11.6" extent="1-16" drill="0.35"/>
+<via x="40.95" y="12.4" extent="1-16" drill="0.35"/>
 </signal>
 <signal name="N$41">
-<via x="18.75" y="10.9" extent="1-16" drill="0.35"/>
+<via x="41.6" y="11.6" extent="1-16" drill="0.35"/>
 </signal>
 <signal name="N$42">
-<via x="19.8" y="10.8" extent="1-16" drill="0.35"/>
-</signal>
-<signal name="N$43">
-<via x="20.85" y="11.55" extent="1-16" drill="0.35"/>
-</signal>
-<signal name="N$44">
-<via x="21.35" y="12.5" extent="1-16" drill="0.35"/>
-</signal>
-<signal name="N$45">
-<via x="21" y="13.5" extent="1-16" drill="0.35"/>
-</signal>
-<signal name="N$46">
-<via x="19.95" y="13.05" extent="1-16" drill="0.35"/>
-</signal>
-<signal name="N$47">
-<via x="19.2" y="12.15" extent="1-16" drill="0.35"/>
+<via x="42.35" y="12.45" extent="1-16" drill="0.35"/>
 </signal>
 </signals>
