File: STM32F413CG/STM32F413CG_WM8731.brd (EAGLE design)
At the start: 54 x 33 mm, 59 parts, among them IC1 STM32F413CGU6, IC2 WM8731SEDS_RV, J2 1503_02, X1 USB-MICROB-SMD

Commit message: added
Parts:
- moved LED2 1.21 mm to (15.0, 18.4)
- moved C8 0.68 mm to (24.9, 12.5)
- moved C38 0.65 mm to (12.5, 17.9)
- moved C5 0.55 mm to (16.0, 6.07)
- moved C12 0.43 mm to (6.56, 16.6)
- moved C14 0.36 mm to (25.9, 3.40)
- moved R2 0.15 mm to (24.5, 7.43)
- moved R5 0.11 mm to (9.38, 8.83)
- moved C20 0.10 mm to (21.8, 2.65)
- moved C6 0.10 mm to (11.6, 14.3)
Routing:
- net N$8: track 15.3 -> 20.9 mm
- net GND: track 272.3 -> 277.8 mm
- net VDD: track 189.9 -> 192.3 mm
- net N$6: track 19.9 -> 17.7 mm
- net B5: track 26.2 -> 24.4 mm
- net A5: track 1.22 -> 2.52 mm
- net B7: track 21.5 -> 20.7 mm
- net B3: track 13.4 -> 14.1 mm
- net N$16: track 47.7 -> 47.0 mm
- net A15: track 13.0 -> 13.7 mm
- net N$48: track 3.55 -> 4.26 mm

Commit message: added
Parts:
- moved C2 0.35 mm to (31.0, 19.9)
- moved C4 0.25 mm to (27.7, 19.8)
Routing:
- net B5: track 24.4 -> 17.0 mm, vias 0 -> 2
- net B10: track 30.6 -> 31.1 mm
