File: STM32F413CG/STM32F413CG_WM8731.sch (EAGLE design)
At the start: 59 parts, among them IC1 STM32F413CGU6, IC2 WM8731SEDS_RV, J2 1503_02, X1 USB-MICROB-SMD

Commit message: adjusted some smd components
Parts:
- IC1: device STM32F413CGU6:STM32F413CGU6 -> STM32F413CG_edited:STM32F413CGU6
Changed lines of the file:
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@@
 </classes>
 <parts>
-<part name="IC1" library="STM32F413CGU6" deviceset="STM32F413CGU6" device=""/>
+<part name="IC1" library="STM32F413CG_edited" deviceset="STM32F413CGU6" device=""/>
 <part name="JP1" library="F405Pill" deviceset="HEADERHOLE" device="-HEADERHOLE"/>
 <part name="C1" library="C0603C104M4RAC7411" deviceset="C0603C104M4RAC7411" device=""/>
