File: CS43L22-CNZ/withAnalog.brd (EAGLE design)
At the start: 48.2 x 28 mm, 55 parts, among them IC1 CS43L22-CNZ, IC2 LP3985IM5-2.5, J2 1503_02

Commit message: added final
Routing:
- net GND: track 0.00 -> 141.7 mm
- net 3.3V: track 0.00 -> 94.3 mm, vias 0 -> 3
- net 2.5V: track 0.00 -> 94.3 mm, vias 0 -> 3
- net N$15: track 0.00 -> 42.8 mm, vias 0 -> 2
- net N$18: track 0.00 -> 32.5 mm, vias 0 -> 2
- net N$11: track 0.00 -> 27.8 mm, vias 0 -> 1
- net N$16: track 0.00 -> 26.9 mm, vias 0 -> 2
- net N$33: track 0.00 -> 26.2 mm
- net N$26: track 0.00 -> 25.6 mm, vias 0 -> 1
- net N$28: track 0.00 -> 24.8 mm
- net N$35: track 0.00 -> 24.5 mm
- net N$9: track 0.00 -> 24.5 mm
- net D4: track 0.00 -> 24.2 mm
- net N$27: track 0.00 -> 22.4 mm
- net N$25: track 0.00 -> 20.3 mm, vias 0 -> 1
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